Commit message: ♥ 없는 의존성 패키지 수정하고 예전 M모델에 호환되게 소스 수정

File: tetra_description/urdf/tetra_bak.xacro (robot description, xacro)
@@ -14,8 +14,8 @@
   </xacro:macro>
    <!-- Include all component files -->
-   <xacro:include filename="$(find tetraDS_description)/urdf/tetraDS/materials.urdf.xacro" />
-   <xacro:include filename="$(find tetraDS_description)/urdf/tetraDS/base.urdf.xacro" />
+   <xacro:include filename="$(find tetra_description)/urdf/materials.urdf.xacro" />
+   <xacro:include filename="$(find tetra_description)/urdf/base.urdf.xacro" />
    <!-- Add the base and wheels -->
-   <base name="base" color="Black"/>
+   <base name="base" color="black"/>
   <link name="laser">
       <visual>
@@ -24,5 +24,5 @@
           <box size="0.01 0.01 0.01" />
         </geometry>
-        <material name="Grey" />
+        <material name="grey" />
       </visual>
   </link>
@@ -38,5 +38,5 @@
           <box size="0.01 0.01 0.01" />
         </geometry>
-        <material name="Grey" />
+        <material name="grey" />
       </visual>
   </link>
@@ -46,5 +46,5 @@
     <child link="imu_link" />
   </joint>
-  <link name="usb_cam">
+  <link name="camera">
       <visual>
         <origin xyz="0 0 0" rpy="0 0 0" />
@@ -52,11 +52,11 @@
           <box size="0.01 0.01 0.01" />
         </geometry>
-        <material name="Grey" />
+        <material name="grey" />
       </visual>
   </link>
-  <joint name="usb_cam" type="fixed">
+  <joint name="camera" type="fixed">
     <origin xyz="-0.384 0.0 0.1387" rpy="1.5708 3.14159 4.71239"/>
     <parent link="base_link"/>
-    <child link="usb_cam" />
+    <child link="camera" />
   </joint>
  <link name="Front_bumper">
@@ -66,5 +66,5 @@
           <box size="0.01 0.48 0.01" />
         </geometry>
-        <material name="TransparentBlack" />
+        <material name="transparentblack" />
       </visual>
   </link>
@@ -80,5 +80,5 @@
           <box size="0.01 0.01 0.01" />
         </geometry>
-        <material name="Grey" />
+        <material name="grey" />
       </visual>
   </link>
@@ -94,5 +94,5 @@
           <box size="0.01 0.01 0.01" />
         </geometry>
-        <material name="Grey" />
+        <material name="grey" />
       </visual>
   </link>
@@ -108,5 +108,5 @@
           <box size="0.01 0.01 0.01" />
         </geometry>
-        <material name="Grey" />
+        <material name="grey" />
       </visual>
   </link>
@@ -122,5 +122,5 @@
           <box size="0.01 0.01 0.01" />
         </geometry>
-        <material name="Grey" />
+        <material name="grey" />
       </visual>
   </link>
@@ -136,5 +136,5 @@
           <box size="0.01 0.01 0.01" />
         </geometry>
-        <material name="Grey" />
+        <material name="grey" />
       </visual>
   </link>
@@ -150,5 +150,5 @@
           <box size="0.01 0.01 0.01" />
         </geometry>
-        <material name="Grey" />
+        <material name="grey" />
       </visual>
   </link>
@@ -158,24 +158,3 @@
     <child link="camera2_link" />
   </joint>
- <link name="base_Upperlink">
-   <visual>
-    <origin xyz=" 0 0 0 " rpy="0 0 0" />
-      <geometry>
-        <mesh
-          filename="package://tetraDS_description/meshes/Platform Body_U.STL" scale="0.001 0.001 0.001" />
-      </geometry>
-      <material name="TransparentRed"/>
-    </visual>
-      <collision>
-            <origin xyz="0 0 0" rpy="0 0 0"/>
-            <geometry>
-                <cylinder length="${base_length}" radius="${base_radius}"/>
-            </geometry>
-      </collision>
-  </link>
-  <joint name="base_Upperlink" type="fixed">
-    <origin xyz="0.0 0.0 0.0" rpy="0 0 0" />
-    <parent link="base_link"/>
-    <child link="base_Upperlink" />
-  </joint>
 </robot>
